File: Hardware/Production/SparkFun Soft Power Switch-Panel.brd (EAGLE design)
At the start: 149.1 x 138.7 mm, 1746 parts, among them J1 Ext Button, J101 System Power, J103 Ext Button, J104 MCU Control, J107 System Power, J109 Ext Button, J11 System Power, J110 MCU Control, J113 System Power, J115 Ext Button, J116 MCU Control, J119 System Power, J121 Ext Button, J122 MCU Control, J125 System Power, J127 Ext Button, J128 MCU Control, J13 Ext Button, J131 System Power, J133 Ext Button, J134 MCU Control, J137 System Power, J139 Ext Button, J14 MCU Control, J140 MCU Control, J143 System Power, J145 Ext Button, J146 MCU Control, J149 System Power, J151 Ext Button, J152 MCU Control, J155 System Power, J157 Ext Button, J158 MCU Control, J161 System Power, J163 Ext Button, J164 MCU Control, J167 System Power, J169 Ext Button, J17 System Power, J170 MCU Control, J173 System Power, J175 Ext Button, J176 MCU Control, J179 System Power, J19 Ext Button, J20 MCU Control, J23 System Power, J25 Ext Button, J26 MCU Control, J29 System Power, J3 Ext Button, J31 Ext Button, J32 MCU Control, J35 System Power, J37 Ext Button, J38 MCU Control, J4 MCU Control, J41 System Power, J43 Ext Button, J44 MCU Control, J47 System Power, J49 Ext Button, J50 MCU Control, J53 System Power, J55 Ext Button, J56 MCU Control, J59 System Power, J6 MCU Control, J61 Ext Button, J62 MCU Control, J65 System Power, J67 Ext Button, J68 MCU Control, J7 System Power, J71 System Power, J73 Ext Button, J74 MCU Control, J77 System Power, J79 Ext Button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

Commit message: x02: Add fast off. Add zener protection. Increase V rating of cap. Increase cap size.
Parts:
- added D61, D64, D67, D70, D73, D76, D79, D82, D85, D88: Power, SparkFun-LED:LED-0603
- added D62, D65, D68, D71, D74, D77, D80, D83, D86, D89: 250mA/100V, SparkFun-DiscreteSemi:SOD-323
- added D63, D66, D69, D72, D75, D78, D81, D84, D87, D90: 3.3V, SparkFun-DiscreteSemi:SOD-323
- added U$841, U$871, U$872, U$902, U$903: (no value), output:#GND#0
- added U$842, U$873, U$904: (no value), output:#SEN#CTRL#1
- added U$843, U$874, U$905: (no value), output:ON#OFF0
- added U$844, U$866, U$875, U$897, U$906, U$928: (no value), output:BATT0
- added U$845, U$867, U$876, U$898, U$907, U$929: (no value), output:SYS1
- added U$846, U$847, U$854, U$856, U$877, U$878, U$885, U$887, U$908, U$909, U$916, U$918: (no value), output:#0
- added U$848, U$849, U$855, U$857, U$879, U$880, U$886, U$888, U$910, U$911, U$917, U$919: (no value), output:#1
- added U$850, U$881, U$912: (no value), output:#MEAS#0
- added U$851, U$882, U$913: (no value), output:SWITCH2
- added U$852, U$864, U$883, U$895, U$914, U$926: (no value), output:ON0
- added U$853, U$884, U$915: (no value), output:#LED#0
- added U$858, U$889, U$920: (no value), output:SOFT0
- added U$859, U$890, U$921: (no value), output:POWER1
- added U$860, U$891, U$922: (no value), output:SWITCH_2
- added U$861, U$892, U$923: (no value), output:SOFT_0
- added U$862, U$893, U$924: (no value), output:POWER_1
- added U$863, U$894, U$925: (no value), output:OFF1
- added U$865, U$896, U$927: (no value), output:#FASTOFF#0
- added U$868, U$899, U$930: SPARKX-LOGO2, SparkX:SPARKX-TINY
- added U$869, U$900: SPARKX-LOGO3, SparkX:SPARKX-SMALL
- added U$870, U$901: (no value), output:#BTN#2
- C10, C13, C16, C19, C22, C25, C28, C3, C31, C34, C37, C40, C43, C46, C49, C52, C55, C58, C61, C64, C67, C7, C70, C73, C76, C79, C82, C85, C88: value 10uF -> 0.1uF
- C12, C15, C18, C21, C24, C27, C30, C33, C36, C39, C42, C45, C48, C51, C54, C57, C6, C60, C63, C66, C69, C72, C75, C78, C81, C84, C87, C9, C90: value 0.1uF -> 22uF; device SparkFun-Capacitors:0603 -> SparkFun-Capacitors:0805
- C4: value 10uF -> 22uF; device SparkFun-Capacitors:0603 -> SparkFun-Capacitors:0805
- D10, D16, D22, D28, D34, D4, D40, D46, D52, D58: value 250mA/100V -> Power; device SparkFun-DiscreteSemi:SOD-323 -> SparkFun-LED:LED-0603
- D11, D17, D23, D29, D35, D41, D47, D5, D53, D59: value Power -> 250mA/100V; device SparkFun-LED:LED-0603 -> SparkFun-DiscreteSemi:SOD-323
- D12, D18, D24, D30, D36, D42, D48, D54, D6, D60: value 250mA/100V -> 3.3V
- D15, D2, D21, D27, D33, D39, D45, D51, D57, D9: value Power -> 3.3V; device SparkFun-LED:LED-0603 -> SparkFun-DiscreteSemi:SOD-323
- J100, J106, J112, J118, J124, J130, J136, J142, J148, J154, J16, J160, J166, J172, J178, J22, J28, J34, J40, J46, J52, J58, J64, J70, J76, J82, J88, J9, J94: value (none) -> System Power
- J101, J107, J11, J113, J119, J125, J131, J137, J143, J149, J155, J161, J167, J17, J173, J179, J23, J29, J35, J41, J47, J53, J59, J65, J71, J77, J83, J89, J95: value System Power -> (none); device SparkFun-Connectors:1X02_NO_SILK -> SparkFun-Connectors:JST-2-SMD
- J102, J108, J114, J12, J120, J126, J132, J138, J144, J150, J156, J162, J168, J174, J18, J180, J24, J30, J36, J42, J48, J54, J60, J66, J72, J78, J84, J90, J96: device SparkFun-Connectors:JST-2-SMD -> SparkFun-Connectors:1X03_NO_SILK
- J104, J110, J116, J122, J128, J134, J14, J140, J146, J152, J158, J164, J170, J176, J20, J26, J32, J38, J44, J50, J56, J62, J68, J74, J80, J86, J92, J98: value MCU Control -> (none); device SparkFun-Connectors:1X02_NO_SILK -> SparkFun-Connectors:JST-2-SMD
- J105, J111, J117, J123, J129, J135, J141, J147, J15, J153, J159, J165, J171, J177, J21, J27, J33, J39, J45, J51, J57, J63, J69, J75, J81, J87, J93, J99: device SparkFun-Connectors:JST-2-SMD -> SparkFun-Connectors:1X02_NO_SILK
- J3: value Ext Button -> (none); device SparkFun-Connectors:1X02_NO_SILK -> SparkFun-Connectors:1X03_NO_SILK
- J4: value MCU Control -> Ext Button
- J6: value MCU Control -> (none)
- R102, R107, R112, R117, R12, R122, R127, R132, R137, R142, R147, R17, R22, R27, R32, R37, R4, R42, R47, R52, R57, R62, R67, R7, R72, R77, R82, R87, R92, R97: value 100k -> 10k
- U$100, U$184: device output:#LED#0 -> output:BATT0
- U$101, U$185, U$318, U$402, U$411, U$495, U$597, U$681: device output:#0 -> output:SYS1
- U$102, U$236, U$298, U$319, U$320, U$382, U$40, U$412, U$48, U$515, U$544, U$599, U$606, U$608, U$692, U$823: device output:#1 -> output:#0
- U$105, U$49, U$609, U$693: device output:SOFT0 -> output:#1
- U$106: device output:POWER1 -> output:#MEAS#0
- U$107: device output:SWITCH_2 -> output:SWITCH2
- U$108: device output:SOFT_0 -> output:ON0
- U$109: device output:POWER_1 -> output:#LED#0
- U$110, U$141, U$474, U$505, U$670, U$701, U$754, U$785: value SPARKX-LOGO3 -> (none); device SparkX:SPARKX-SMALL -> output:#0
- U$111, U$167, U$671, U$755: device output:OFF1 -> output:#1
- U$112, U$196, U$267, U$351, U$420, U$575, U$71, U$784: device output:ON0 -> output:#0
- U$113, U$166, U$197, U$390, U$421, U$446, U$477, U$82: value SPARKX-LOGO3 -> (none); device SparkX:SPARKX-SMALL -> output:#1
- U$114: device output:#BTN#2 -> output:SOFT0
- U$115, U$704: device output:#GND#0 -> output:POWER1
- U$116, U$395: device output:#GND#0 -> output:SWITCH_2
- U$117: device output:#SEN#CTRL#1 -> output:SOFT_0
- U$118: device output:ON#OFF0 -> output:POWER_1
- U$119: device output:BATT0 -> output:OFF1
- U$120, U$232: device output:SYS1 -> output:ON0
- U$121, U$493, U$710, U$803: device output:#0 -> output:#FASTOFF#0
- U$122, U$131, U$215, U$317, U$38, U$401, U$689, U$773: device output:#0 -> output:BATT0
- U$123, U$132, U$216, U$39, U$628, U$690, U$712, U$774: device output:#1 -> output:SYS1
- U$124, U$186, U$403, U$496: value (none) -> SPARKX-LOGO2; device output:#1 -> SparkX:SPARKX-TINY
- U$125: value (none) -> SPARKX-LOGO3; device output:#MEAS#0 -> SparkX:SPARKX-SMALL
- U$126: device output:SWITCH2 -> output:#BTN#2
- U$127, U$252, U$407, U$840: device output:ON0 -> output:#GND#0
- U$128, U$716: device output:#LED#0 -> output:#GND#0
- U$129, U$346, U$439, U$625: device output:#0 -> output:#SEN#CTRL#1
- U$130, U$347, U$440, U$68: device output:#1 -> output:ON#OFF0
- U$133, U$329, U$413, U$637: device output:SOFT0 -> output:#0
- U$134, U$358, U$50, U$722: device output:POWER1 -> output:#0
- U$135, U$359, U$415, U$51: device output:SWITCH_2 -> output:#1
- U$136, U$640, U$724, U$80: device output:SOFT_0 -> output:#1
- U$137: device output:POWER_1 -> output:#MEAS#0
- U$138, U$169: value SPARKX-LOGO3 -> (none); device SparkX:SPARKX-SMALL -> output:SWITCH2
- U$139: device output:OFF1 -> output:ON0
- U$140, U$295: device output:ON0 -> output:#LED#0
- U$142, U$198, U$702, U$786: device output:#BTN#2 -> output:#1
- U$143, U$172, U$227, U$451, U$536, U$732, U$815, U$816: device output:#GND#0 -> output:#0
- U$144, U$228, U$423, U$452, U$507, U$508, U$731, U$787: device output:#GND#0 -> output:#1
- U$145: device output:#SEN#CTRL#1 -> output:SOFT0
- U$146: device output:ON#OFF0 -> output:POWER1
- U$147: device output:BATT0 -> output:SWITCH_2
- U$148: device output:SYS1 -> output:SOFT_0
- U$149, U$521, U$738, U$831: device output:#0 -> output:POWER_1
- U$15, U$558, U$589: value SPARKX-LOGO3 -> SPARKX-LOGO2; device SparkX:SPARKX-SMALL -> SparkX:SPARKX-TINY
- U$150, U$243, U$429, U$801: device output:#0 -> output:OFF1
- U$151, U$244, U$263, U$356, U$46, U$740, U$802: device output:#1 -> output:ON0
- U$152, U$214, U$431, U$524: device output:#1 -> output:#FASTOFF#0
- U$153, U$69: device output:#MEAS#0 -> output:BATT0
- U$154, U$70: device output:SWITCH2 -> output:SYS1
- U$155: value (none) -> SPARKX-LOGO2; device output:ON0 -> SparkX:SPARKX-TINY
- U$156: value (none) -> SPARKX-LOGO3; device output:#LED#0 -> SparkX:SPARKX-SMALL
- U$157, U$374, U$467, U$653: device output:#0 -> output:#BTN#2
- U$158, U$375, U$376, U$438, U$468, U$655, U$748, U$96: device output:#1 -> output:#GND#0
- U$159, U$345, U$437, U$65, U$654, U$66, U$717, U$747: device output:#0 -> output:#GND#0
- U$160, U$656, U$67, U$718: device output:#1 -> output:#SEN#CTRL#1
- U$161: device output:SOFT0 -> output:ON#OFF0
- U$162, U$246: device output:POWER1 -> output:BATT0
- U$163, U$247: device output:SWITCH_2 -> output:SYS1
- U$164, U$360, U$444, U$668: device output:SOFT_0 -> output:#0
- U$165, U$389, U$753, U$81: device output:POWER_1 -> output:#0
- U$168, U$323: device output:ON0 -> output:#MEAS#0
- U$170, U$58: device output:#BTN#2 -> output:ON0
- U$171, U$760: device output:#GND#0 -> output:#LED#0
- U$173, U$229, U$733, U$817: device output:#SEN#CTRL#1 -> output:#1
- U$174, U$258, U$482: device output:ON#OFF0 -> output:#0
- U$175, U$259, U$483, U$539: device output:BATT0 -> output:#1
- U$176: device output:SYS1 -> output:SOFT0
- U$177, U$549, U$766: device output:#0 -> output:POWER1
- U$178, U$271, U$457, U$829: device output:#0 -> output:SWITCH_2
- U$179, U$272, U$768, U$830: device output:#1 -> output:SOFT_0
- U$180, U$242, U$459, U$552: device output:#1 -> output:POWER_1
- U$181: device output:#MEAS#0 -> output:OFF1
- U$182, U$294: device output:SWITCH2 -> output:ON0
- U$183: device output:ON0 -> output:#FASTOFF#0
- U$187, U$373, U$745, U$94: value (none) -> SPARKX-LOGO3; device output:#0 -> SparkX:SPARKX-SMALL
- U$188, U$684, U$746, U$95: device output:#1 -> output:#BTN#2
- U$189, U$469: device output:SOFT0 -> output:#GND#0
- U$190, U$778: device output:POWER1 -> output:#GND#0
- U$191: device output:SWITCH_2 -> output:#SEN#CTRL#1
- U$192: device output:SOFT_0 -> output:ON#OFF0
- U$193, U$277: device output:POWER_1 -> output:BATT0
- U$194, U$225, U$278, U$309: value SPARKX-LOGO3 -> (none); device SparkX:SPARKX-SMALL -> output:SYS1
- U$195, U$391, U$475, U$699: device output:OFF1 -> output:#0
- U$199, U$788: device output:#GND#0 -> output:#MEAS#0
- U$200, U$479: device output:#GND#0 -> output:SWITCH2
- U$201, U$89: device output:#SEN#CTRL#1 -> output:ON0
- U$202: device output:ON#OFF0 -> output:#LED#0
- U$203, U$567, U$763: device output:BATT0 -> output:#0
- U$204, U$260, U$764: device output:SYS1 -> output:#1
- U$206, U$290, U$297, U$299, U$353, U$383, U$485, U$514, U$569, U$570, U$607, U$663, U$73, U$793: device output:#0 -> output:#1
- U$207, U$300, U$796: device output:#1 -> output:SOFT0
- U$208, U$270, U$487, U$580: device output:#1 -> output:POWER1
- U$209: device output:#MEAS#0 -> output:SWITCH_2
- U$210: device output:SWITCH2 -> output:SOFT_0
- U$211, U$56: device output:ON0 -> output:POWER_1
- U$212: device output:#LED#0 -> output:OFF1
- U$213, U$325, U$430, U$523, U$542, U$635, U$709, U$821: device output:#0 -> output:ON0
- U$217: value (none) -> SPARKX-LOGO2; device output:SOFT0 -> SparkX:SPARKX-TINY
- U$218: value (none) -> SPARKX-LOGO3; device output:POWER1 -> SparkX:SPARKX-SMALL
- U$219: device output:SWITCH_2 -> output:#BTN#2
- U$220, U$500: device output:SOFT_0 -> output:#GND#0
- U$221, U$809: device output:POWER_1 -> output:#GND#0
- U$222, U$253: value SPARKX-LOGO3 -> (none); device SparkX:SPARKX-SMALL -> output:#SEN#CTRL#1
- U$223: device output:OFF1 -> output:ON#OFF0
- U$224, U$308, U$379, U$463: device output:ON0 -> output:BATT0
- U$226, U$422, U$506, U$730: device output:#BTN#2 -> output:#0
- U$230: device output:ON#OFF0 -> output:#MEAS#0
- U$231: device output:BATT0 -> output:SWITCH2
- U$233, U$47, U$605, U$822: device output:#0 -> output:#LED#0
- U$237, U$321, U$545, U$601: device output:#MEAS#0 -> output:#1
- U$238: device output:SWITCH2 -> output:SOFT0
- U$239, U$84: device output:ON0 -> output:POWER1
- U$240: device output:#LED#0 -> output:SWITCH_2
- U$241, U$458, U$551, U$737: device output:#0 -> output:SOFT_0
- U$245: device output:SOFT0 -> output:#FASTOFF#0
- U$248: value (none) -> SPARKX-LOGO2; device output:SOFT_0 -> SparkX:SPARKX-TINY
- U$249: value (none) -> SPARKX-LOGO3; device output:POWER_1 -> SparkX:SPARKX-SMALL
- U$250, U$281: value SPARKX-LOGO3 -> (none); device SparkX:SPARKX-SMALL -> output:#BTN#2
- U$251, U$531: device output:OFF1 -> output:#GND#0
- U$254: device output:#BTN#2 -> output:ON#OFF0
- U$255, U$339, U$60: device output:#GND#0 -> output:BATT0
- U$256, U$31, U$340, U$535, U$619: device output:#GND#0 -> output:SYS1
- U$257, U$453, U$537, U$761: device output:#SEN#CTRL#1 -> output:#0
- U$26, U$586, U$617: value SPARKX-LOGO3 -> (none); device SparkX:SPARKX-SMALL -> output:#FASTOFF#0
- U$261, U$633, U$75: device output:#0 -> output:#MEAS#0
- U$262, U$355, U$45, U$541: device output:#0 -> output:SWITCH2
- U$264, U$326, U$543, U$636: device output:#1 -> output:#LED#0
- U$265, U$41, U$629, U$825: device output:#MEAS#0 -> output:#0
- U$266, U$322, U$42, U$826: device output:SWITCH2 -> output:#1
- U$268, U$352, U$576, U$632: device output:#LED#0 -> output:#1
- U$269, U$486, U$579, U$765: device output:#0 -> output:SOFT0
- U$273: device output:SOFT0 -> output:POWER_1
- U$274: device output:POWER1 -> output:OFF1
- U$275, U$387: device output:SWITCH_2 -> output:ON0
- U$276: device output:SOFT_0 -> output:#FASTOFF#0
- U$279: value (none) -> SPARKX-LOGO2; device output:OFF1 -> SparkX:SPARKX-TINY
- U$280, U$435: value (none) -> SPARKX-LOGO3; device output:ON0 -> SparkX:SPARKX-SMALL
- U$282, U$562: device output:#BTN#2 -> output:#GND#0
- U$284, U$563: device output:#GND#0 -> output:#SEN#CTRL#1
- U$285: device output:#SEN#CTRL#1 -> output:ON#OFF0
- U$286, U$370: device output:ON#OFF0 -> output:BATT0
- U$287, U$371: device output:BATT0 -> output:SYS1
- U$288, U$484, U$568, U$792: device output:SYS1 -> output:#0
- U$29, U$534, U$618: device output:#BTN#2 -> output:BATT0
- U$292, U$354, U$571, U$664: device output:#1 -> output:#MEAS#0
- U$293: device output:#MEAS#0 -> output:SWITCH2
- U$296, U$660, U$72: device output:#LED#0 -> output:#0
- U$301: device output:SOFT0 -> output:POWER1
- U$302: device output:POWER1 -> output:SWITCH_2
- U$303: device output:SWITCH_2 -> output:SOFT_0
- U$304: device output:SOFT_0 -> output:POWER_1
- U$305: device output:POWER_1 -> output:OFF1
- U$306, U$337, U$418, U$449: value SPARKX-LOGO3 -> (none); device SparkX:SPARKX-SMALL -> output:ON0
- U$307: device output:OFF1 -> output:#FASTOFF#0
- U$310: value (none) -> SPARKX-LOGO2; device output:#BTN#2 -> SparkX:SPARKX-TINY
- U$311, U$32: value (none) -> SPARKX-LOGO3; device output:#GND#0 -> SparkX:SPARKX-SMALL
- U$312, U$591: device output:#GND#0 -> output:#BTN#2
- U$313, U$593: device output:#SEN#CTRL#1 -> output:#GND#0
- U$314, U$34: device output:ON#OFF0 -> output:#GND#0
- U$315: device output:BATT0 -> output:#SEN#CTRL#1
- U$316: device output:SYS1 -> output:ON#OFF0
- U$324: device output:#LED#0 -> output:SWITCH2
- U$33: device output:#SEN#CTRL#1 -> output:#BTN#2
- U$330, U$414, U$638, U$694: device output:POWER1 -> output:#1
- U$331: device output:SWITCH_2 -> output:SOFT0
- U$332: device output:SOFT_0 -> output:POWER1
- U$333: device output:POWER_1 -> output:SWITCH_2
- U$334, U$365: value SPARKX-LOGO3 -> (none); device SparkX:SPARKX-SMALL -> output:SOFT_0
- U$335: device output:OFF1 -> output:POWER_1
- U$336, U$491: device output:ON0 -> output:OFF1
- U$338: device output:#BTN#2 -> output:#FASTOFF#0
- U$341: value (none) -> SPARKX-LOGO2; device output:#SEN#CTRL#1 -> SparkX:SPARKX-TINY
- U$342: value (none) -> SPARKX-LOGO3; device output:ON#OFF0 -> SparkX:SPARKX-SMALL
- U$343: device output:BATT0 -> output:#BTN#2
- U$344, U$624: device output:SYS1 -> output:#GND#0
- U$348, U$410, U$432, U$494, U$627, U$711, U$720, U$804: device output:#1 -> output:BATT0
- U$349, U$433: device output:#MEAS#0 -> output:SYS1
- U$35, U$623: device output:BATT0 -> output:#GND#0
- U$350, U$546, U$630: device output:SWITCH2 -> output:#0
- U$357: device output:SOFT0 -> output:#LED#0
- U$36: device output:SYS1 -> output:#SEN#CTRL#1
- U$361, U$445, U$669, U$725: device output:POWER_1 -> output:#1
- U$362, U$393: value SPARKX-LOGO3 -> (none); device SparkX:SPARKX-SMALL -> output:SOFT0
- U$363: device output:OFF1 -> output:POWER1
- U$364, U$519: device output:ON0 -> output:SWITCH_2
- U$366: device output:#BTN#2 -> output:POWER_1
- U$367, U$88: device output:#GND#0 -> output:OFF1
- U$368, U$480, U$647, U$759: device output:#GND#0 -> output:ON0
- U$369: device output:#SEN#CTRL#1 -> output:#FASTOFF#0
- U$37, U$409, U$626, U$719: device output:#0 -> output:ON#OFF0
- U$372: value (none) -> SPARKX-LOGO2; device output:SYS1 -> SparkX:SPARKX-TINY
- U$377: device output:#MEAS#0 -> output:#SEN#CTRL#1
- U$378: device output:SWITCH2 -> output:ON#OFF0
- U$380, U$464: device output:#LED#0 -> output:SYS1
- U$385: device output:SOFT0 -> output:#MEAS#0
- U$386: device output:POWER1 -> output:SWITCH2
- U$388: device output:SOFT_0 -> output:#LED#0
- U$392, U$43, U$476, U$547, U$631, U$700, U$756: device output:ON0 -> output:#1
- U$394: device output:#BTN#2 -> output:POWER1
- U$396, U$675: device output:#GND#0 -> output:SOFT_0
- U$397: device output:#SEN#CTRL#1 -> output:POWER_1
- U$398: device output:ON#OFF0 -> output:OFF1
- U$399, U$511: device output:BATT0 -> output:ON0
- U$400: device output:SYS1 -> output:#FASTOFF#0
- U$404, U$466, U$683, U$776: value (none) -> SPARKX-LOGO3; device output:#1 -> SparkX:SPARKX-SMALL
- U$405: device output:#MEAS#0 -> output:#BTN#2
- U$406, U$686: device output:SWITCH2 -> output:#GND#0
- U$408: device output:#LED#0 -> output:#SEN#CTRL#1
- U$416: device output:SOFT_0 -> output:#MEAS#0
- U$417: device output:POWER_1 -> output:SWITCH2
- U$419: device output:OFF1 -> output:#LED#0
- U$424, U$703: device output:#GND#0 -> output:SOFT0
- U$425: device output:#SEN#CTRL#1 -> output:POWER1
- U$426: device output:ON#OFF0 -> output:SWITCH_2
- U$427: device output:BATT0 -> output:SOFT_0
- U$428: device output:SYS1 -> output:POWER_1
- U$434: value (none) -> SPARKX-LOGO2; device output:SWITCH2 -> SparkX:SPARKX-TINY
- U$436: device output:#LED#0 -> output:#BTN#2
- U$44: device output:#LED#0 -> output:#MEAS#0
- U$441, U$525: device output:SOFT0 -> output:BATT0
- U$442, U$526: device output:POWER1 -> output:SYS1
- U$443, U$639, U$723, U$79: device output:SWITCH_2 -> output:#0
- U$447: device output:OFF1 -> output:#MEAS#0
- U$448, U$603: device output:ON0 -> output:SWITCH2
- U$450: device output:#BTN#2 -> output:#LED#0
- U$454, U$538, U$762, U$818: device output:ON#OFF0 -> output:#1
- U$455: device output:BATT0 -> output:SOFT0
- U$456: device output:SYS1 -> output:POWER1
- U$460, U$522, U$739, U$832: device output:#1 -> output:OFF1
- U$461, U$573: device output:#MEAS#0 -> output:ON0
- U$462: device output:SWITCH2 -> output:#FASTOFF#0
- U$465, U$682, U$775, U$93: value (none) -> SPARKX-LOGO2; device output:#0 -> SparkX:SPARKX-TINY
- U$470: device output:POWER1 -> output:#SEN#CTRL#1
- U$471: device output:SWITCH_2 -> output:ON#OFF0
- U$472, U$556: device output:SOFT_0 -> output:BATT0
- U$473, U$557: device output:POWER_1 -> output:SYS1
- U$478: device output:#BTN#2 -> output:#MEAS#0
- U$481: device output:#SEN#CTRL#1 -> output:#LED#0
- U$488, U$550, U$767: device output:#1 -> output:SWITCH_2
- U$489: device output:#MEAS#0 -> output:SOFT_0
- U$490: device output:SWITCH2 -> output:POWER_1
- U$492, U$604: device output:#LED#0 -> output:ON0
- U$497: value (none) -> SPARKX-LOGO3; device output:SOFT0 -> SparkX:SPARKX-SMALL
- U$498: device output:POWER1 -> output:#BTN#2
- U$499, U$779: device output:SWITCH_2 -> output:#GND#0
- U$501: device output:POWER_1 -> output:#SEN#CTRL#1
- U$502, U$533: value SPARKX-LOGO3 -> (none); device SparkX:SPARKX-SMALL -> output:ON#OFF0
- U$503, U$587: device output:OFF1 -> output:BATT0
- U$504, U$588, U$659, U$743: device output:ON0 -> output:SYS1
- U$509: device output:#SEN#CTRL#1 -> output:#MEAS#0
- U$510: device output:ON#OFF0 -> output:SWITCH2
- U$512: device output:SYS1 -> output:#LED#0
- U$517: device output:#MEAS#0 -> output:SOFT0
- U$518: device output:SWITCH2 -> output:POWER1
- U$52: device output:SOFT_0 -> output:SOFT0
- U$520: device output:#LED#0 -> output:SOFT_0
- U$527: value (none) -> SPARKX-LOGO2; device output:SWITCH_2 -> SparkX:SPARKX-TINY
- U$528: value (none) -> SPARKX-LOGO3; device output:SOFT_0 -> SparkX:SPARKX-SMALL
- U$529: device output:POWER_1 -> output:#BTN#2
- U$53: device output:POWER_1 -> output:POWER1
- U$530, U$561, U$810: value SPARKX-LOGO3 -> (none); device SparkX:SPARKX-SMALL -> output:#GND#0
- U$532, U$687: device output:ON0 -> output:#SEN#CTRL#1
- U$54, U$85: value SPARKX-LOGO3 -> (none); device SparkX:SPARKX-SMALL -> output:SWITCH_2
- U$540: device output:SYS1 -> output:#MEAS#0
- U$548: device output:#LED#0 -> output:SOFT0
- U$55: device output:OFF1 -> output:SOFT_0
- U$553: device output:SOFT0 -> output:OFF1
- U$554, U$666: device output:POWER1 -> output:ON0
- U$555: device output:SWITCH_2 -> output:#FASTOFF#0
- U$559: value (none) -> SPARKX-LOGO3; device output:OFF1 -> SparkX:SPARKX-SMALL
- U$560, U$715: device output:ON0 -> output:#BTN#2
- U$564: device output:#GND#0 -> output:ON#OFF0
- U$565, U$649: device output:#SEN#CTRL#1 -> output:BATT0
- U$566, U$650: device output:ON#OFF0 -> output:SYS1
- U$57: value SPARKX-LOGO3 -> (none); device SparkX:SPARKX-SMALL -> output:OFF1
- U$572, U$634, U$76: device output:#1 -> output:SWITCH2
- U$574: device output:SWITCH2 -> output:#LED#0
- U$581: device output:SOFT0 -> output:SWITCH_2
- U$582: device output:POWER1 -> output:SOFT_0
- U$583: device output:SWITCH_2 -> output:POWER_1
- U$584: device output:SOFT_0 -> output:OFF1
- U$585, U$697: device output:POWER_1 -> output:ON0
- U$59, U$648: device output:#GND#0 -> output:#FASTOFF#0
- U$590: value (none) -> SPARKX-LOGO3; device output:#BTN#2 -> SparkX:SPARKX-SMALL
- U$594: device output:ON#OFF0 -> output:#SEN#CTRL#1
- U$595: device output:BATT0 -> output:ON#OFF0
- U$596, U$680: device output:SYS1 -> output:BATT0
- U$602: device output:SWITCH2 -> output:#MEAS#0
- U$61: device output:#SEN#CTRL#1 -> output:SYS1
- U$610: device output:POWER1 -> output:SOFT0
- U$611: device output:SWITCH_2 -> output:POWER1
- U$612: device output:SOFT_0 -> output:SWITCH_2
- U$613: device output:POWER_1 -> output:SOFT_0
- U$614, U$645: value SPARKX-LOGO3 -> (none); device SparkX:SPARKX-SMALL -> output:POWER_1
- U$62: value (none) -> SPARKX-LOGO2; device output:ON#OFF0 -> SparkX:SPARKX-TINY
- U$620: value (none) -> SPARKX-LOGO2; device output:#GND#0 -> SparkX:SPARKX-TINY
- U$621: value (none) -> SPARKX-LOGO3; device output:#SEN#CTRL#1 -> SparkX:SPARKX-SMALL
- U$622: device output:ON#OFF0 -> output:#BTN#2
- U$63: value (none) -> SPARKX-LOGO3; device output:BATT0 -> SparkX:SPARKX-SMALL
- U$64: device output:SYS1 -> output:#BTN#2
- U$641: device output:POWER_1 -> output:SOFT0
- U$642, U$673: value SPARKX-LOGO3 -> (none); device SparkX:SPARKX-SMALL -> output:POWER1
- U$643: device output:OFF1 -> output:SWITCH_2
- U$644, U$799: device output:ON0 -> output:SOFT_0
- U$646: device output:#BTN#2 -> output:OFF1
- U$651: value (none) -> SPARKX-LOGO2; device output:BATT0 -> SparkX:SPARKX-TINY
- U$652: value (none) -> SPARKX-LOGO3; device output:SYS1 -> SparkX:SPARKX-SMALL
- U$657: device output:#MEAS#0 -> output:ON#OFF0
- U$658, U$742: device output:SWITCH2 -> output:BATT0
- U$665: device output:SOFT0 -> output:SWITCH2
- U$667: device output:SWITCH_2 -> output:#LED#0
- U$672, U$827: device output:ON0 -> output:SOFT0
- U$674: device output:#BTN#2 -> output:SWITCH_2
- U$676, U$87: device output:#GND#0 -> output:POWER_1
- U$677: device output:#SEN#CTRL#1 -> output:OFF1
- U$678, U$790: device output:ON#OFF0 -> output:ON0
- U$679: device output:BATT0 -> output:#FASTOFF#0
- U$685, U$97: device output:#MEAS#0 -> output:#GND#0
- U$688: device output:#LED#0 -> output:ON#OFF0
- U$695: device output:SWITCH_2 -> output:#MEAS#0
- U$696: device output:SOFT_0 -> output:SWITCH2
- U$698, U$729: value SPARKX-LOGO3 -> (none); device SparkX:SPARKX-SMALL -> output:#LED#0
- U$705: device output:#SEN#CTRL#1 -> output:SWITCH_2
- U$706: device output:ON#OFF0 -> output:SOFT_0
- U$707: device output:BATT0 -> output:POWER_1
- U$708: device output:SYS1 -> output:OFF1
- U$713: value (none) -> SPARKX-LOGO2; device output:#MEAS#0 -> SparkX:SPARKX-TINY
- U$714: value (none) -> SPARKX-LOGO3; device output:SWITCH2 -> SparkX:SPARKX-SMALL
- U$721, U$805: device output:SOFT0 -> output:SYS1
- U$726, U$757: value SPARKX-LOGO3 -> (none); device SparkX:SPARKX-SMALL -> output:#MEAS#0
- U$727: device output:OFF1 -> output:SWITCH2
- U$734: device output:ON#OFF0 -> output:SOFT0
- U$735: device output:BATT0 -> output:POWER1
- U$736: device output:SYS1 -> output:SWITCH_2
- U$741: device output:#MEAS#0 -> output:#FASTOFF#0
- U$744: value (none) -> SPARKX-LOGO2; device output:#LED#0 -> SparkX:SPARKX-TINY
- U$749: device output:SOFT0 -> output:#SEN#CTRL#1
- U$750: device output:POWER1 -> output:ON#OFF0
- U$751, U$835: device output:SWITCH_2 -> output:BATT0
- U$752, U$836: device output:SOFT_0 -> output:SYS1
- U$758: device output:#BTN#2 -> output:SWITCH2
- U$769: device output:#MEAS#0 -> output:POWER_1
- U$77, U$833: device output:SOFT0 -> output:ON0
- U$770: device output:SWITCH2 -> output:OFF1
- U$772: device output:#LED#0 -> output:#FASTOFF#0
- U$777: device output:SOFT0 -> output:#BTN#2
- U$78: device output:POWER1 -> output:#LED#0
- U$780: device output:SOFT_0 -> output:#SEN#CTRL#1
- U$781: device output:POWER_1 -> output:ON#OFF0
- U$782, U$813: value SPARKX-LOGO3 -> (none); device SparkX:SPARKX-SMALL -> output:BATT0
- U$783: device output:OFF1 -> output:SYS1
- U$789: device output:#SEN#CTRL#1 -> output:SWITCH2
- U$791: device output:BATT0 -> output:#LED#0
- U$797: device output:#MEAS#0 -> output:POWER1
- U$798: device output:SWITCH2 -> output:SWITCH_2
- U$800: device output:#LED#0 -> output:POWER_1
- U$806: value (none) -> SPARKX-LOGO2; device output:POWER1 -> SparkX:SPARKX-TINY
- U$807: value (none) -> SPARKX-LOGO3; device output:SWITCH_2 -> SparkX:SPARKX-SMALL
- U$808: device output:SOFT_0 -> output:#BTN#2
- U$811: device output:OFF1 -> output:#SEN#CTRL#1
- U$812, U$99: device output:ON0 -> output:ON#OFF0
- U$814: device output:#BTN#2 -> output:SYS1
- U$819: device output:BATT0 -> output:#MEAS#0
- U$820: device output:SYS1 -> output:SWITCH2
- U$828: device output:#LED#0 -> output:POWER1
- U$83: device output:OFF1 -> output:SOFT0
- U$834: device output:POWER1 -> output:#FASTOFF#0
- U$837: value (none) -> SPARKX-LOGO2; device output:POWER_1 -> SparkX:SPARKX-TINY
- U$839: device output:OFF1 -> output:#BTN#2
- U$86: device output:#BTN#2 -> output:SOFT_0
- U$90: device output:ON#OFF0 -> output:#FASTOFF#0
- U$98: device output:SWITCH2 -> output:#SEN#CTRL#1
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Connections:
- removed net N$121: D49.C, R121.2
- removed net N$122: C73.2, Q25.G1, R123.1
- removed net N$123: C74.1, C75.2, Q25.D1, Q25.G2, R124.1
- removed net N$124: D49.A, JP49.1
- removed net N$125: C74.2, JP50.2
- removed net N$126: D51.C, R126.2
- removed net N$127: C76.2, Q26.G1, R128.1
- removed net N$128: C77.1, C78.2, Q26.D1, Q26.G2, R129.1
- removed net N$129: D51.A, JP51.1
- removed net N$130: C77.2, JP52.2
- removed net N$131: D53.C, R131.2
- removed net N$132: C79.2, Q27.G1, R133.1
- removed net N$133: C80.1, C81.2, Q27.D1, Q27.G2, R134.1
- removed net N$134: D53.A, JP53.1
- removed net N$135: C80.2, JP54.2
- removed net N$136: D55.C, R136.2
- removed net N$137: C82.2, Q28.G1, R138.1
- removed net N$138: C83.1, C84.2, Q28.D1, Q28.G2, R139.1
- removed net N$139: D55.A, JP55.1
- removed net N$140: C83.2, JP56.2
- removed net N$141: D57.C, R141.2
- removed net N$142: C85.2, Q29.G1, R143.1
- removed net N$143: C86.1, C87.2, Q29.D1, Q29.G2, R144.1
- removed net N$144: D57.A, JP57.1
- removed net N$145: C86.2, JP58.2
- removed net N$146: D59.C, R146.2
- removed net N$147: C88.2, Q30.G1, R148.1
- removed net N$148: C89.1, C90.2, Q30.D1, Q30.G2, R149.1
- removed net N$149: D59.A, JP59.1
- removed net N$150: C89.2, JP60.2
- new net FAST_OFF: C4.2, J3.2, Q1.G1, R5.1
- new net FAST_OFF1: C6.2, J12.2, Q2.G1, R8.1
- new net FAST_OFF10: C33.2, J66.2, Q11.G1, R53.1
- new net FAST_OFF11: C36.2, J72.2, Q12.G1, R58.1
- new net FAST_OFF12: C39.2, J78.2, Q13.G1, R63.1
- new net FAST_OFF13: C42.2, J84.2, Q14.G1, R68.1
- new net FAST_OFF14: C45.2, J90.2, Q15.G1, R73.1
- new net FAST_OFF15: C48.2, J96.2, Q16.G1, R78.1
- new net FAST_OFF16: C51.2, J102.2, Q17.G1, R83.1
- new net FAST_OFF17: C54.2, J108.2, Q18.G1, R88.1
- new net FAST_OFF18: C57.2, J114.2, Q19.G1, R93.1
- new net FAST_OFF19: C60.2, J120.2, Q20.G1, R98.1
- new net FAST_OFF2: C9.2, J18.2, Q3.G1, R13.1
- new net FAST_OFF20: C63.2, J126.2, Q21.G1, R103.1
- new net FAST_OFF21: C66.2, J132.2, Q22.G1, R108.1
- new net FAST_OFF22: C69.2, J138.2, Q23.G1, R113.1
- new net FAST_OFF23: C72.2, J144.2, Q24.G1, R118.1
- new net FAST_OFF24: C75.2, J150.2, Q25.G1, R123.1
- new net FAST_OFF25: C78.2, J156.2, Q26.G1, R128.1
- new net FAST_OFF26: C81.2, J162.2, Q27.G1, R133.1
- new net FAST_OFF27: C84.2, J168.2, Q28.G1, R138.1
- new net FAST_OFF28: C87.2, J174.2, Q29.G1, R143.1
- new net FAST_OFF29: C90.2, J180.2, Q30.G1, R148.1
- new net FAST_OFF3: C12.2, J24.2, Q4.G1, R18.1
- new net FAST_OFF4: C15.2, J30.2, Q5.G1, R23.1
- new net FAST_OFF5: C18.2, J36.2, Q6.G1, R28.1
- new net FAST_OFF6: C21.2, J42.2, Q7.G1, R33.1
- new net FAST_OFF7: C24.2, J48.2, Q8.G1, R38.1
- new net FAST_OFF8: C27.2, J54.2, Q9.G1, R43.1
- new net FAST_OFF9: C30.2, J60.2, Q10.G1, R48.1
- net GND: now also D2.A, J3.1; no longer J6.2
- net GND1: now also D6.A, J11.1, J6.2; no longer J11.2, J3.2
- net GND10: now also D33.A, J62.1, J63.2, J65.1; no longer J62.2, J63.1, J65.2
- net GND11: now also D36.A, J68.1, J69.2, J71.1; no longer J68.2, J69.1, J71.2
- net GND12: now also D39.A, J74.1, J75.2, J77.1; no longer J74.2, J75.1, J77.2
- net GND13: now also D42.A, J80.1, J81.2, J83.1; no longer J80.2, J81.1, J83.2
- net GND14: now also D45.A, J86.1, J87.2, J89.1; no longer J86.2, J87.1, J89.2
- net GND15: now also D48.A, J92.1, J93.2, J95.1; no longer J92.2, J93.1, J95.2
- net GND16: now also D51.A, J101.1, J98.1, J99.2; no longer J101.2, J98.2, J99.1
- net GND17: now also D54.A, J104.1, J105.2, J107.1; no longer J104.2, J105.1, J107.2
- net GND18: now also D57.A, J110.1, J111.2, J113.1; no longer J110.2, J111.1, J113.2
- net GND19: now also D60.A, J116.1, J117.2, J119.1; no longer J116.2, J117.1, J119.2
- net GND2: now also D9.A, J14.1, J15.2, J17.1; no longer J14.2, J15.1, J17.2
- net GND20: now also D63.A, J122.1, J123.2, J125.1; no longer J122.2, J123.1, J125.2
- net GND21: now also D66.A, J128.1, J129.2, J131.1; no longer J128.2, J129.1, J131.2
- net GND22: now also D69.A, J134.1, J135.2, J137.1; no longer J134.2, J135.1, J137.2
- net GND23: now also D72.A, J140.1, J141.2, J143.1; no longer J140.2, J141.1, J143.2
- net GND24: now also D75.A, J146.1, J147.2, J149.1; no longer J146.2, J147.1, J149.2
- net GND25: now also D78.A, J152.1, J153.2, J155.1; no longer J152.2, J153.1, J155.2
- net GND26: now also D81.A, J158.1, J159.2, J161.1; no longer J158.2, J159.1, J161.2
- net GND27: now also D84.A, J164.1, J165.2, J167.1; no longer J164.2, J165.1, J167.2
- net GND28: now also D87.A, J170.1, J171.2, J173.1; no longer J170.2, J171.1, J173.2
- net GND29: now also D90.A, J176.1, J177.2, J179.1; no longer J176.2, J177.1, J179.2
- net GND3: now also D12.A, J20.1, J21.2, J23.1; no longer J20.2, J21.1, J23.2
- net GND4: now also D15.A, J26.1, J27.2, J29.1; no longer J26.2, J27.1, J29.2
- net GND5: now also D18.A, J32.1, J33.2, J35.1; no longer J32.2, J33.1, J35.2
- net GND6: now also D21.A, J38.1, J39.2, J41.1; no longer J38.2, J39.1, J41.2
- net GND7: now also D24.A, J44.1, J45.2, J47.1; no longer J44.2, J45.1, J47.2
- net GND8: now also D27.A, J50.1, J51.2, J53.1; no longer J50.2, J51.1, J53.2
- net GND9: now also D30.A, J56.1, J57.2, J59.1; no longer J56.2, J57.1, J59.2
- net N$10: now also D7.A, JP5.1; no longer D5.C, R11.2
- net N$100: now also C73.2, JP50.2; no longer C59.2, JP40.2
- net N$101: now also D76.C, R126.2; no longer D41.C, R101.2
- net N$102: now also C76.1, C77.2, Q26.D1, Q26.G2, R129.1; no longer C61.2, Q21.G1, R103.1
- net N$103: now also D76.A, JP51.1; no longer C62.1, C63.2, Q21.D1, Q21.G2, R104.1
- net N$104: now also C76.2, JP52.2; no longer D41.A, JP41.1
- net N$105: now also D79.C, R131.2; no longer C62.2, JP42.2
- net N$106: now also C79.1, C80.2, Q27.D1, Q27.G2, R134.1; no longer D43.C, R106.2
- net N$107: now also D79.A, JP53.1; no longer C64.2, Q22.G1, R108.1
- net N$108: now also C79.2, JP54.2; no longer C65.1, C66.2, Q22.D1, Q22.G2, R109.1
- net N$109: now also D82.C, R136.2; no longer D43.A, JP43.1
- net N$11: now also JP6.2; no longer Q3.G1, R13.1
- net N$110: now also C82.1, C83.2, Q28.D1, Q28.G2, R139.1; no longer C65.2, JP44.2
- net N$111: now also D82.A, JP55.1; no longer D45.C, R111.2
- net N$112: now also C82.2, JP56.2; no longer C67.2, Q23.G1, R113.1
- net N$113: now also D85.C, R141.2; no longer C68.1, C69.2, Q23.D1, Q23.G2, R114.1
- net N$114: now also C85.1, C86.2, Q29.D1, Q29.G2, R144.1; no longer D45.A, JP45.1
- net N$115: now also D85.A, JP57.1; no longer C68.2, JP46.2
- net N$116: now also C85.2, JP58.2; no longer D47.C, R116.2
- net N$117: now also D88.C, R146.2; no longer C70.2, Q24.G1, R118.1
- net N$118: now also C88.1, C89.2, Q30.D1, Q30.G2, R149.1; no longer C71.1, C72.2, Q24.D1, Q24.G2, R119.1
- net N$119: now also D88.A, JP59.1; no longer D47.A, JP47.1
- net N$12: now also D10.C, R16.2; no longer C8.1, C9.2, Q3.D1, Q3.G2, R14.1
- net N$120: now also C88.2, JP60.2; no longer C71.2, JP48.2
- net N$13: now also C10.1, C11.2, Q4.D1, Q4.G2, R19.1; no longer D5.A, JP5.1
- net N$14: now also D10.A, JP7.1; no longer C8.2, JP6.2
- net N$16: now also C10.2, JP8.2; no longer D7.C, R16.2
- net N$17: now also D13.C, R21.2; no longer C10.2, Q4.G1, R18.1
- net N$18: now also C13.1, C14.2, Q5.D1, Q5.G2, R24.1; no longer C11.1, C12.2, Q4.D1, Q4.G2, R19.1
- net N$19: now also D13.A, JP9.1; no longer D7.A, JP7.1
- net N$20: now also C13.2, JP10.2; no longer C11.2, JP8.2
- net N$21: now also D16.C, R26.2; no longer D9.C, R21.2
- net N$22: now also C16.1, C17.2, Q6.D1, Q6.G2, R29.1; no longer C13.2, Q5.G1, R23.1
- net N$23: now also D16.A, JP11.1; no longer C14.1, C15.2, Q5.D1, Q5.G2, R24.1
- net N$24: now also C16.2, JP12.2; no longer D9.A, JP9.1
- net N$25: now also D19.C, R31.2; no longer C14.2, JP10.2
- net N$26: now also C19.1, C20.2, Q7.D1, Q7.G2, R34.1; no longer D11.C, R26.2
- net N$27: now also D19.A, JP13.1; no longer C16.2, Q6.G1, R28.1
- net N$28: now also C19.2, JP14.2; no longer C17.1, C18.2, Q6.D1, Q6.G2, R29.1
- net N$29: now also D22.C, R36.2; no longer D11.A, JP11.1
- net N$3: now also D4.C; no longer D2.C
- net N$30: now also C22.1, C23.2, Q8.D1, Q8.G2, R39.1; no longer C17.2, JP12.2
- net N$31: now also D22.A, JP15.1; no longer D13.C, R31.2
- net N$32: now also C22.2, JP16.2; no longer C19.2, Q7.G1, R33.1
- net N$33: now also D25.C, R41.2; no longer C20.1, C21.2, Q7.D1, Q7.G2, R34.1
- net N$34: now also C25.1, C26.2, Q9.D1, Q9.G2, R44.1; no longer D13.A, JP13.1
- net N$35: now also D25.A, JP17.1; no longer C20.2, JP14.2
- net N$36: now also C25.2, JP18.2; no longer D15.C, R36.2
- net N$37: now also D28.C, R46.2; no longer C22.2, Q8.G1, R38.1
- net N$38: now also C28.1, C29.2, Q10.D1, Q10.G2, R49.1; no longer C23.1, C24.2, Q8.D1, Q8.G2, R39.1
- net N$39: now also D28.A, JP19.1; no longer D15.A, JP15.1
- net N$4: now also C3.1, C5.2, Q2.D1, Q2.G2, R9.1; no longer C4.2, Q2.G1, R8.1
- net N$40: now also C28.2, JP20.2; no longer C23.2, JP16.2
- net N$41: now also D31.C, R51.2; no longer D17.C, R41.2
- net N$42: now also C31.1, C32.2, Q11.D1, Q11.G2, R54.1; no longer C25.2, Q9.G1, R43.1
- net N$43: now also D31.A, JP21.1; no longer C26.1, C27.2, Q9.D1, Q9.G2, R44.1
- net N$44: now also C31.2, JP22.2; no longer D17.A, JP17.1
- net N$45: now also D34.C, R56.2; no longer C26.2, JP18.2
- net N$46: now also C34.1, C35.2, Q12.D1, Q12.G2, R59.1; no longer D19.C, R46.2
- net N$47: now also D34.A, JP23.1; no longer C28.2, Q10.G1, R48.1
- net N$48: now also C34.2, JP24.2; no longer C29.1, C30.2, Q10.D1, Q10.G2, R49.1
- net N$49: now also D37.C, R61.2; no longer D19.A, JP19.1
- net N$5: now also D4.A, JP3.1; no longer C5.1, C6.2, Q2.D1, Q2.G2, R9.1
- net N$50: now also C37.1, C38.2, Q13.D1, Q13.G2, R64.1; no longer C29.2, JP20.2
- net N$51: now also D37.A, JP25.1; no longer D21.C, R51.2
- net N$52: now also C37.2, JP26.2; no longer C31.2, Q11.G1, R53.1
- net N$53: now also D40.C, R66.2; no longer C32.1, C33.2, Q11.D1, Q11.G2, R54.1
- net N$54: now also C40.1, C41.2, Q14.D1, Q14.G2, R69.1; no longer D21.A, JP21.1
- net N$55: now also D40.A, JP27.1; no longer C32.2, JP22.2
- net N$56: now also C40.2, JP28.2; no longer D23.C, R56.2
- net N$57: now also D43.C, R71.2; no longer C34.2, Q12.G1, R58.1
- net N$58: now also C43.1, C44.2, Q15.D1, Q15.G2, R74.1; no longer C35.1, C36.2, Q12.D1, Q12.G2, R59.1
- net N$59: now also D43.A, JP29.1; no longer D23.A, JP23.1
- net N$60: now also C43.2, JP30.2; no longer C35.2, JP24.2
- net N$61: now also D46.C, R76.2; no longer D25.C, R61.2
- net N$62: now also C46.1, C47.2, Q16.D1, Q16.G2, R79.1; no longer C37.2, Q13.G1, R63.1
- net N$63: now also D46.A, JP31.1; no longer C38.1, C39.2, Q13.D1, Q13.G2, R64.1
- net N$64: now also C46.2, JP32.2; no longer D25.A, JP25.1
- net N$65: now also D49.C, R81.2; no longer C38.2, JP26.2
- net N$66: now also C49.1, C50.2, Q17.D1, Q17.G2, R84.1; no longer D27.C, R66.2
- net N$67: now also D49.A, JP33.1; no longer C40.2, Q14.G1, R68.1
- net N$68: now also C49.2, JP34.2; no longer C41.1, C42.2, Q14.D1, Q14.G2, R69.1
- net N$69: now also D52.C, R86.2; no longer D27.A, JP27.1
- net N$7: now also C3.2, JP4.2; no longer D2.A, JP3.1
- net N$70: now also C52.1, C53.2, Q18.D1, Q18.G2, R89.1; no longer C41.2, JP28.2
- net N$71: now also D52.A, JP35.1; no longer D29.C, R71.2
- net N$72: now also C52.2, JP36.2; no longer C43.2, Q15.G1, R73.1
- net N$73: now also D55.C, R91.2; no longer C44.1, C45.2, Q15.D1, Q15.G2, R74.1
- net N$74: now also C55.1, C56.2, Q19.D1, Q19.G2, R94.1; no longer D29.A, JP29.1
- net N$75: now also D55.A, JP37.1; no longer C44.2, JP30.2
- net N$76: now also C55.2, JP38.2; no longer D31.C, R76.2
- net N$77: now also D58.C, R96.2; no longer C46.2, Q16.G1, R78.1
- net N$78: now also C58.1, C59.2, Q20.D1, Q20.G2, R99.1; no longer C47.1, C48.2, Q16.D1, Q16.G2, R79.1
- net N$79: now also D58.A, JP39.1; no longer D31.A, JP31.1
- net N$8: now also D7.C, R11.2; no longer C3.2, Q1.G1, R5.1
- net N$80: now also C58.2, JP40.2; no longer C47.2, JP32.2
- net N$81: now also D61.C, R101.2; no longer D33.C, R81.2
- net N$82: now also C61.1, C62.2, Q21.D1, Q21.G2, R104.1; no longer C49.2, Q17.G1, R83.1
- net N$83: now also D61.A, JP41.1; no longer C50.1, C51.2, Q17.D1, Q17.G2, R84.1
- net N$84: now also C61.2, JP42.2; no longer D33.A, JP33.1
- net N$85: now also D64.C, R106.2; no longer C50.2, JP34.2
- net N$86: now also C64.1, C65.2, Q22.D1, Q22.G2, R109.1; no longer D35.C, R86.2
- net N$87: now also D64.A, JP43.1; no longer C52.2, Q18.G1, R88.1
- net N$88: now also C64.2, JP44.2; no longer C53.1, C54.2, Q18.D1, Q18.G2, R89.1
- net N$89: now also D67.C, R111.2; no longer D35.A, JP35.1
- net N$9: now also C7.1, C8.2, Q3.D1, Q3.G2, R14.1; no longer C5.2, JP4.2
- net N$90: now also C67.1, C68.2, Q23.D1, Q23.G2, R114.1; no longer C53.2, JP36.2
- net N$91: now also D67.A, JP45.1; no longer D37.C, R91.2
- net N$92: now also C67.2, JP46.2; no longer C55.2, Q19.G1, R93.1
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Routing:
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Other:
- board text added: "x02"
- board text removed: "x01"

Commit message: Replace MOSFET on panel.
Parts:
- Q1, Q10, Q11, Q12, Q13, Q14, Q15, Q16, Q17, Q18, Q19, Q2, Q20, Q21, Q22, Q23, Q24, Q25, Q26, Q27, Q28, Q29, Q3, Q30, Q4, Q5, Q6, Q7, Q8, Q9: value DMC2700UDM -> SIL2308-TP
