File: Hardware/SparkFun Soft Power Switch.brd (EAGLE design)
At the start: 25.4 x 20.3 mm, 59 parts, among them J1 Ext Button, J6 MCU Control, J7 System Power, Q1 DMC2700UDM

Commit message: x02: Add fast off. Add zener protection. Increase V rating of cap. Increase cap size.
Parts:
- removed C3: 10uF, SparkFun-Capacitors:0603
- removed J6: MCU Control, SparkFun-Connectors:1X02_NO_SILK
- added C4: 22uF, SparkFun-Capacitors:0805
- added D2: 3.3V, SparkFun-DiscreteSemi:SOD-323
- added J3: (no value), SparkFun-Connectors:1X03_NO_SILK
- added U$26: (no value), output:#FASTOFF#0
- added U$29: (no value), output:BATT0
- added U$31: (no value), output:SYS1
- R4: value 100k -> 10k
- U$15: value SPARKX-LOGO3 -> SPARKX-LOGO2; device SparkX:SPARKX-SMALL -> SparkX:SPARKX-TINY
- moved U$5 2.54 mm to (6.35, 6.22)
- moved U$15 1.57 mm to (5.97, 5.46)
- moved D3 1.27 mm to (11.0, 3.81)
- moved U$10 0.89 mm to (17.8, 7.87)
- moved U$11 0.76 mm to (17.7, 12.3)
- moved U$12 0.76 mm to (7.75, 7.75)
- moved U$9 0.63 mm to (7.75, 12.4)
Connections:
- removed net N$8: C3.2, Q1.G1, R5.1
- new net FAST_OFF: C4.2, J3.2, Q1.G1, R5.1
- net GND: now also D2.A, J3.1; no longer J6.2
- net POWER_SENSE/CTRL: now also D2.C, J3.3; no longer J6.1
- net VCC: now also C4.1; no longer C3.1
Routing:
- net FAST_OFF: track 0.00 -> 15.9 mm, vias 0 -> 1
- net N$8: track 7.77 -> 0.00 mm
- net POWER_SENSE/CTRL: track 6.40 -> 8.25 mm
- net POWER_BTN: track 34.1 -> 32.8 mm
Other:
- board text added: "x02"
- board text removed: "x01"

Commit message: Replace MOSFET with SIL2308-TP
Parts:
- Q1: value DMC2700UDM -> SIL2308-TP
Changed lines of the file:
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@@
 <layer number="47" name="Measures" color="7" fill="1" visible="no" active="yes"/>
 <layer number="48" name="Document" color="7" fill="1" visible="no" active="yes"/>
-<layer number="49" name="Reference" color="7" fill="1" visible="yes" active="yes"/>
+<layer number="49" name="Reference" color="7" fill="1" visible="no" active="yes"/>
 <layer number="50" name="dxf" color="7" fill="1" visible="no" active="yes"/>
 <layer number="51" name="tDocu" color="6" fill="1" visible="yes" active="yes"/>
@@
 <attribute name="VALUE" x="14.3891" y="17.7546" size="0.6096" layer="27" font="vector" ratio="20" rot="R270" align="top-center"/>
 </element>
-<element name="Q1" library="SparkFun-DiscreteSemi" package="SOT26" value="DMC2700UDM" x="12.7" y="10.16" smashed="yes">
+<element name="Q1" library="SparkFun-DiscreteSemi" package="SOT26" value="SIL2308-TP" x="12.7" y="10.16" smashed="yes">
 <attribute name="NAME" x="12.7" y="11.938" size="0.6096" layer="25" font="vector" ratio="20" align="bottom-center"/>
-<attribute name="PROD_ID" value="TRANS-11993" x="7.62" y="16.51" size="1.778" layer="27" font="vector" ratio="15" display="off"/>
+<attribute name="PROD_ID" value="TRANS-15717" x="7.62" y="16.51" size="1.778" layer="27" font="vector" ratio="15" display="off"/>
 <attribute name="VALUE" x="12.7" y="8.382" size="0.6096" layer="27" font="vector" ratio="20" align="top-center"/>
 </element>

Commit message: Add prod ID to power LED.
Parts:
- D1: value Power -> RED
Changed lines of the file:
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@@
 <attribute name="VALUE" value="1k" x="18.034" y="17.78" size="0.6096" layer="27" font="vector" ratio="20" rot="R270" align="top-center"/>
 </element>
-<element name="D1" library="SparkFun-LED" package="LED-0603" value="Power" x="17.78" y="17.78" smashed="yes" rot="R270">
+<element name="D1" library="SparkFun-LED" package="LED-0603" value="RED" x="17.78" y="17.78" smashed="yes" rot="R270">
 <attribute name="NAME" x="21.1709" y="17.78" size="0.6096" layer="25" font="vector" ratio="20" rot="R270" align="bottom-center"/>
-<attribute name="VALUE" x="14.3891" y="17.7546" size="0.6096" layer="27" font="vector" ratio="20" rot="R270" align="top-center"/>
+<attribute name="PROD_ID" value="DIO-00819" x="17.78" y="17.78" size="1.778" layer="27" rot="R270" display="off"/>
+<attribute name="VALUE" value="RED" x="14.3891" y="17.7546" size="0.6096" layer="27" font="vector" ratio="20" rot="R270" align="top-center"/>
 </element>
 <element name="Q1" library="SparkFun-DiscreteSemi" package="SOT26" value="SIL2308-TP" x="12.7" y="10.16" smashed="yes">
