File: Hardware/SparkFun Soft Power Switch.sch (EAGLE design)
At the start: 34 parts, among them J1 Ext Button, J7 System Power, Q1 SIL2308-TP

Commit message: Add prod ID to power LED.
Parts:
- D1: value Power -> RED; device SparkFun-LED:LED0603 -> SparkFun-LED:LED-RED0603
Changed lines of the file:
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@@
 <part name="H3" library="SparkFun-Hardware" deviceset="STAND-OFF" device=""/>
 <part name="R2" library="SparkFun-Resistors" deviceset="1KOHM" device="-0603-1/10W-1%" value="1k"/>
-<part name="D1" library="SparkFun-LED" deviceset="LED" device="0603" value="Power"/>
+<part name="D1" library="SparkFun-LED" deviceset="LED-RED" device="0603" value="RED"/>
 <part name="Q1" library="SparkFun-DiscreteSemi" deviceset="MOSFET_COMPLIMENTARY_PAIR" device="-SIL2308" value="SIL2308-TP"/>
 <part name="R4" library="SparkFun-Resistors" deviceset="10KOHM" device="-0603-1/10W-1%" value="10k"/>
@@
 <attribute name="VALUE" x="164.084" y="101.6" size="1.778" layer="96" font="vector" rot="R90" align="top-center"/>
 </instance>
-<instance part="D1" gate="D1" x="162.56" y="114.3" smashed="yes">
+<instance part="D1" gate="G$1" x="162.56" y="114.3" smashed="yes">
 <attribute name="NAME" x="159.131" y="109.728" size="1.778" layer="95" font="vector" rot="R90"/>
 <attribute name="VALUE" x="164.465" y="109.728" size="1.778" layer="96" font="vector" rot="R90" align="top-left"/>
@@
 <wire x1="162.56" y1="109.22" x2="162.56" y2="106.68" width="0.1524" layer="91"/>
 <pinref part="R2" gate="G$1" pin="2"/>
-<pinref part="D1" gate="D1" pin="C"/>
+<pinref part="D1" gate="G$1" pin="C"/>
 </segment>
 </net>
@@
 <segment>
 <pinref part="JP1" gate="G$1" pin="1"/>
-<pinref part="D1" gate="D1" pin="A"/>
+<pinref part="D1" gate="G$1" pin="A"/>
 <wire x1="162.56" y1="119.38" x2="162.56" y2="116.84" width="0.1524" layer="91"/>
 </segment>

Commit message: Add 12VGS max note
Other:
- note added: "VGS Max 12V"
Changed lines of the file:
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@@
 immediately turn off the system.</text>
 <wire x1="99.06" y1="144.78" x2="109.22" y2="127.762" width="0.2032" layer="97"/>
+<text x="137.16" y="133.604" size="1.778" layer="97">VGS Max 12V</text>
 </plain>
 <instances>
